Commit message: add launch files for rviz and gazebo

File: mybot_description/urdf/mybot.urdf.xacro (robot description, xacro)
@@ -5,8 +5,18 @@
     <xacro:property name="effort" value="30.0" />
     <xacro:property name="velocity" value="10.0" />
+    <!-- create intertia macro -->
+    <xacro:macro name="default_inertia" params="mass">
+        <inertial>
+            <mass value="${mass}" />
+            <inertia ixx="1.0" ixy="0.0" ixz="0.0"
+                iyy="1.0" iyz="0.0"
+                izz="1.0" />
+        </inertial>
+    </xacro:macro>
     <!-- link world-->
     <link name="world" />
     <!-- base link -->
     <link name="base_link">
+        <xacro:default_inertia mass="1.0" />
         <visual>
             <!-- this will define the position and orientation of mesh w.r.t to base_link-->
@@ -17,4 +27,8 @@
             </geometry>
         </visual>
+        <collision>
+            <mesh filename="package://mybot_description/meshes/basement.STL"
+                scale="0.01 0.01 0.01" />
+        </collision>
     </link>
     <!-- fixed joint btw world and base link -->
@@ -27,4 +41,5 @@
     <!-- base_plate link -->
     <link name="base_plate">
+        <xacro:default_inertia mass="0.1" />
         <visual>
             <!-- this will define the position and orientation of mesh w.r.t to base_plate-->
@@ -35,4 +50,8 @@
             </geometry>
         </visual>
+        <collision>
+            <mesh filename="package://mybot_description/meshes/base_plate.STL"
+                scale="0.01 0.01 0.01" />
+        </collision>
     </link>
     <!-- joint btw base_plate and base_link -->
@@ -47,4 +66,5 @@
     <!-- forward drive arm link -->
     <link name="forward_drive_arm">
+        <xacro:default_inertia mass="0.1" />
         <visual>
             <!-- this will define the position and orientation of mesh w.r.t to forward_drive_arm-->
@@ -55,4 +75,8 @@
             </geometry>
         </visual>
+        <collision>
+            <mesh filename="package://mybot_description/meshes/forward_drive_arm.STL"
+                scale="0.01 0.01 0.01" />
+        </collision>
     </link>
     <!-- joint btw the base_plate link and forward_drive_arm link -->
@@ -68,4 +92,5 @@
     <!-- horizontal arm link -->
     <link name="horizontal_arm">
+        <xacro:default_inertia mass="0.1" />
         <visual>
             <!-- this will define the position and orientation of mesh w.r.t to horizontal_arm-->
@@ -76,4 +101,8 @@
             </geometry>
         </visual>
+        <collision>
+            <mesh filename="package://mybot_description/meshes/horizontal_arm.STL"
+                scale="0.01 0.01 0.01" />
+        </collision>
     </link>
     <!-- joint btw the forward_drive_arm link and the horizontal_arm link -->
@@ -90,4 +119,5 @@
     <!-- claw_support link -->
     <link name="claw_support">
+        <xacro:default_inertia mass="0.05" />
         <visual>
             <!-- this will define the position and orientation of mesh w.r.t to claw_support-->
@@ -98,4 +128,8 @@
             </geometry>
         </visual>
+        <collision>
+            <mesh filename="package://mybot_description/meshes/claw_support.STL"
+                scale="0.01 0.01 0.01" />
+        </collision>
     </link>
     <!-- fixed joint btw the the horizontal_arm link  and claw_support link -->
@@ -108,4 +142,5 @@
     <!-- gripper right link -->
     <link name="gripper_right">
+        <xacro:default_inertia mass="0.01" />
         <visual>
             <!-- this will define the position and orientation of mesh w.r.t to gripper_right-->
@@ -116,4 +151,8 @@
             </geometry>
         </visual>
+        <collision>
+            <mesh filename="package://mybot_description/meshes/right_finger.STL"
+                scale="0.01 0.01 0.01" />
+        </collision>
     </link>
     <!-- joint btw the claw_support link and gripper_right -->
@@ -128,4 +167,5 @@
     <!-- gripper left link -->
     <link name="gripper_left">
+        <xacro:default_inertia mass="0.01" />
         <visual>
             <!-- this will define the position and orientation of mesh w.r.t to gripper_left -->
@@ -136,4 +176,8 @@
             </geometry>
         </visual>
+        <collision>
+            <mesh filename="package://mybot_description/meshes/left_finger.STL"
+                scale="0.01 0.01 0.01" />
+        </collision>
     </link>
     <!-- joint btw the claw_support link and gripper_right -->

Commit message: bug fix: collision tag not defined correctly

File: mybot_description/urdf/mybot.urdf.xacro (robot description, xacro)
@@ -1,17 +1,29 @@
 <?xml version="1.0"?>
 <robot xmlns:xacro="http://www.ros.org/wiki/xacro" name="mybot">
+    <!-- Include xacro File
+    <xacro:include filename="$(find mybot_description)/urdf/mybot_gazebo.xacro" />
+    <xacro:include filename="$(find mybot_description)/urdf/mybot_ros2_control.xacro" /> -->
     <!--  xacro properties -->
     <xacro:property name="PI" value="3.14159" />
     <xacro:property name="effort" value="30.0" />
     <xacro:property name="velocity" value="10.0" />
-    <!-- create intertia macro -->
+    <!-- create inertia macro -->
     <xacro:macro name="default_inertia" params="mass">
         <inertial>
             <mass value="${mass}" />
-            <inertia ixx="1.0" ixy="0.0" ixz="0.0"
+            <inertia ixx="1.0" ixy="0.0"
                 iyy="1.0" iyz="0.0"
-                izz="1.0" />
+                izz="1.0" ixz="0.0" />
         </inertial>
     </xacro:macro>
+    <!-- <xacro:macro name="default_transmission" params="joint_no">
+        <transmission name="transmission_${joint_no}">
+            <plugin>transmission_interface/SimpleTransmission</plugin>
+            <joint name="joint_${joint_no}" role="joint1">
+                <mechanicalReduction>1.0</mechanicalReduction>
+            </joint>
+            <actuator name="motor_${joint_no}" role="actuator1" />
+        </transmission>
+    </xacro:macro> -->
     <!-- link world-->
     <link name="world" />
@@ -28,6 +40,9 @@
         </visual>
         <collision>
-            <mesh filename="package://mybot_description/meshes/basement.STL"
-                scale="0.01 0.01 0.01" />
+            <origin xyz="-0.5 -0.5 0.0" rpy="0.0 0.0 0.0" />
+            <geometry>
+                <mesh filename="package://mybot_description/meshes/basement.STL"
+                    scale="0.01 0.01 0.01" />
+            </geometry>
         </collision>
     </link>
@@ -51,6 +66,9 @@
         </visual>
         <collision>
-            <mesh filename="package://mybot_description/meshes/base_plate.STL"
-                scale="0.01 0.01 0.01" />
+            <origin xyz="-0.39 -0.39 -0.56" rpy="0.0 0.0 0.0" />
+            <geometry>
+                <mesh filename="package://mybot_description/meshes/base_plate.STL"
+                    scale="0.01 0.01 0.01" />
+            </geometry>
         </collision>
     </link>
@@ -76,6 +94,9 @@
         </visual>
         <collision>
-            <mesh filename="package://mybot_description/meshes/forward_drive_arm.STL"
-                scale="0.01 0.01 0.01" />
+            <origin xyz="0.19 0.06 -0.08" rpy="0.0 -${PI/2} ${PI/2}" />
+            <geometry>
+                <mesh filename="package://mybot_description/meshes/forward_drive_arm.STL"
+                    scale="0.01 0.01 0.01" />
+            </geometry>
         </collision>
     </link>
@@ -102,6 +123,9 @@
         </visual>
         <collision>
-            <mesh filename="package://mybot_description/meshes/horizontal_arm.STL"
-                scale="0.01 0.01 0.01" />
+            <origin xyz="-0.03 -0.04 -0.06" rpy="${PI/2} 0.0 ${PI/2}" />
+            <geometry>
+                <mesh filename="package://mybot_description/meshes/horizontal_arm.STL"
+                    scale="0.01 0.01 0.01" />
+            </geometry>
         </collision>
     </link>
@@ -129,6 +153,9 @@
         </visual>
         <collision>
-            <mesh filename="package://mybot_description/meshes/claw_support.STL"
-                scale="0.01 0.01 0.01" />
+            <origin xyz="0.0 -0.05 -0.15" rpy="0.0 0.0 ${PI/2}" />
+            <geometry>
+                <mesh filename="package://mybot_description/meshes/claw_support.STL"
+                    scale="0.01 0.01 0.01" />
+            </geometry>
         </collision>
     </link>
@@ -152,6 +179,9 @@
         </visual>
         <collision>
-            <mesh filename="package://mybot_description/meshes/right_finger.STL"
-                scale="0.01 0.01 0.01" />
+            <origin xyz="-0.1 0.5 -0.1" rpy="0.0 0.0 -${PI/2}" />
+            <geometry>
+                <mesh filename="package://mybot_description/meshes/right_finger.STL"
+                    scale="0.01 0.01 0.01" />
+            </geometry>
         </collision>
     </link>
@@ -177,6 +207,9 @@
         </visual>
         <collision>
-            <mesh filename="package://mybot_description/meshes/left_finger.STL"
-                scale="0.01 0.01 0.01" />
+            <origin xyz="-0.04 0.5 -0.1" rpy="0.0 0.0 -${PI/2}" />
+            <geometry>
+                <mesh filename="package://mybot_description/meshes/left_finger.STL"
+                    scale="0.01 0.01 0.01" />
+            </geometry>
         </collision>
     </link>
@@ -193,3 +226,8 @@
         <mimic joint="joint_4" multiplier="-1" />
     </joint>
+    <!-- added transmission to movable joints for gazebo/physics simulation
+    <xacro:default_transmission joint_no="1" />
+    <xacro:default_transmission joint_no="2" />
+    <xacro:default_transmission joint_no="3" />
+    <xacro:default_transmission joint_no="4" /> -->
 </robot>
